Commit message: Updated script

File: RBT_kuka.urdf (robot description, URDF)
Before this commit: robot Robot, 11 links, 10 joints
Links:
- link iiwa_link_0: geometry collision mesh filename=C:\Program Files\MATLAB\R2025b\toolbox\robotics\robotmodels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 scale=1.00000000 1.00000000 1.00000000; visual mesh filename=C:\Program Files\MATLAB\R2025b\toolbox\robotics\robotmodels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 scale=1.00000000 1.00000000 1.00000000
- link iiwa_link_1: geometry collision mesh filename=C:\Program Files\MATLAB\R2025b\toolbox\robotics\robotmodels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 scale=1.00000000 1.00000000 1.00000000; visual mesh filename=C:\Program Files\MATLAB\R2025b\toolbox\robotics\robotmodels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 scale=1.00000000 1.00000000 1.00000000
- link iiwa_link_2: geometry collision mesh filename=C:\Program Files\MATLAB\R2025b\toolbox\robotics\robotmodels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 scale=1.00000000 1.00000000 1.00000000; visual mesh filename=C:\Program Files\MATLAB\R2025b\toolbox\robotics\robotmodels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 scale=1.00000000 1.00000000 1.00000000
- link iiwa_link_3: geometry collision mesh filename=C:\Program Files\MATLAB\R2025b\toolbox\robotics\robotmodels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 scale=1.00000000 1.00000000 1.00000000; visual mesh filename=C:\Program Files\MATLAB\R2025b\toolbox\robotics\robotmodels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 scale=1.00000000 1.00000000 1.00000000
- link iiwa_link_4: geometry collision mesh filename=C:\Program Files\MATLAB\R2025b\toolbox\robotics\robotmodels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 scale=1.00000000 1.00000000 1.00000000; visual mesh filename=C:\Program Files\MATLAB\R2025b\toolbox\robotics\robotmodels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 scale=1.00000000 1.00000000 1.00000000
- link iiwa_link_5: geometry collision mesh filename=C:\Program Files\MATLAB\R2025b\toolbox\robotics\robotmodels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 scale=1.00000000 1.00000000 1.00000000; visual mesh filename=C:\Program Files\MATLAB\R2025b\toolbox\robotics\robotmodels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 scale=1.00000000 1.00000000 1.00000000
- link iiwa_link_6: geometry collision mesh filename=C:\Program Files\MATLAB\R2025b\toolbox\robotics\robotmodels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 scale=1.00000000 1.00000000 1.00000000; visual mesh filename=C:\Program Files\MATLAB\R2025b\toolbox\robotics\robotmodels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 scale=1.00000000 1.00000000 1.00000000
- link iiwa_link_7: geometry collision mesh filename=C:\Program Files\MATLAB\R2025b\toolbox\robotics\robotmodels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 scale=1.00000000 1.00000000 1.00000000; visual mesh filename=C:\Program Files\MATLAB\R2025b\toolbox\robotics\robotmodels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 scale=1.00000000 1.00000000 1.00000000
Joints:
- joint iiwa_joint_5: origin xyz=0.00000000 0.21000000 0.00000000 rpy=1.57079633 -0.00000000 -3.14159265 -> xyz=0.00000000 0.21000000 0.00000000 rpy=1.57079633 -0.00000000  3.14159265
- joint iiwa_joint_7: origin xyz=0.00000000 0.08100000 0.06070000 rpy=1.57079633 -0.00000000 -3.14159265 -> xyz=0.00000000 0.08100000 0.06070000 rpy=1.57079633 -0.00000000  3.14159265
